Commit message: Added new branch catatron_mesh

File: src/notspot_description/urdf/notspot.urdf (robot description, URDF)
Before this commit: robot notspot, 17 links, 16 joints
Links:
- link FL1: mass 0.15334 -> 0.34; geometry collision mesh filename=/home/sudharsan/Documents/notspot_sim_py/src/notspot_descri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; visual mesh filename=/home/sudharsan/Documents/notspot_sim_py/src/notspot_descri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
- link FL2: mass 0.15106 -> 0.084; geometry collision mesh filename=/home/sudharsan/Documents/notspot_sim_py/src/notspot_descri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; visual mesh filename=/home/sudharsan/Documents/notspot_sim_py/src/notspot_descri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
- link FL3: mass 0.023372 -> 0.034; geometry collision mesh filename=/home/sudharsan/Documents/notspot_sim_py/src/notspot_descri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; visual mesh filename=/home/sudharsan/Documents/notspot_sim_py/src/notspot_descri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
- link FL4: mass 0.0391 -> 0.010; geometry collision box size=0.011 0.011 0.011; visual sphere radius=0.001
- link FR1: mass 0.15379 -> 0.233; geometry collision mesh filename=/home/sudharsan/Documents/notspot_sim_py/src/notspot_descri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; visual mesh filename=/home/sudharsan/Documents/notspot_sim_py/src/notspot_descri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
- link FR2: mass 0.15106 -> 0.184; geometry collision mesh filename=/home/sudharsan/Documents/notspot_sim_py/src/notspot_descri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; visual mesh filename=/home/sudharsan/Documents/notspot_sim_py/src/notspot_descri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
- link FR3: mass 0.023372 -> 0.034; geometry collision mesh filename=/home/sudharsan/Documents/notspot_sim_py/src/notspot_descri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; visual mesh filename=/home/sudharsan/Documents/notspot_sim_py/src/notspot_descri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
- link FR4: mass 0.0391 -> 0.010; geometry collision box size=0.011 0.011 0.011; visual sphere radius=0.001
- link RL1: mass 0.15379 -> 0.233; geometry collision mesh filename=/home/sudharsan/Documents/notspot_sim_py/src/notspot_descri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; visual mesh filename=/home/sudharsan/Documents/notspot_sim_py/src/notspot_descri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
- link RL2: mass 0.15106 -> 0.084; geometry collision mesh filename=/home/sudharsan/Documents/notspot_sim_py/src/notspot_descri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; visual mesh filename=/home/sudharsan/Documents/notspot_sim_py/src/notspot_descri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
- link RL3: mass 0.023372 -> 0.034; geometry collision mesh filename=/home/sudharsan/Documents/notspot_sim_py/src/notspot_descri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; visual mesh filename=/home/sudharsan/Documents/notspot_sim_py/src/notspot_descri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
- link RL4: mass 0.0391 -> 0.010; geometry collision box size=0.011 0.011 0.011; visual sphere radius=0.001
- link RR1: mass 0.15379 -> 0.233; geometry collision mesh filename=/home/sudharsan/Documents/notspot_sim_py/src/notspot_descri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; visual mesh filename=/home/sudharsan/Documents/notspot_sim_py/src/notspot_descri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
- link RR2: mass 0.15106 -> 0.084; geometry collision mesh filename=/home/sudharsan/Documents/notspot_sim_py/src/notspot_descri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; visual mesh filename=/home/sudharsan/Documents/notspot_sim_py/src/notspot_descri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
- link RR3: mass 0.023372 -> 0.034; geometry collision mesh filename=/home/sudharsan/Documents/notspot_sim_py/src/notspot_descri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; visual mesh filename=/home/sudharsan/Documents/notspot_sim_py/src/notspot_descri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
- link RR4: mass 0.0391 -> 0.010; geometry collision box size=0.011 0.011 0.011; visual sphere radius=0.001
- link base_link: mass 0.81776 -> 0.81700; geometry collision mesh filename=/home/sudharsan/Documents/notspot_sim_py/src/notspot_descri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; visual mesh filename=/home/sudharsan/Documents/notspot_sim_py/src/notspot_descri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
Joints:
- joint FL1_joint: axis 0 0 1 -> 1.000 0.000 0.000; limit lower=-3 upper=3 effort=${effort_limit} velocity=3 -> lower=-0.78540 upper=1.57080 effort=1.4 velocity=1.04720; origin xyz=0.0954 0.04 0 rpy=1.5708 0 -1.5708 -> xyz=0.09170 0.05355 -0.00279
- joint FL2_joint: axis 0 0 1 -> 0.000 1.000 0.000; limit lower=-3 upper=3 effort=${effort_limit} velocity=3 -> lower=0.00020 upper=2.35619 effort=1.4 velocity=1.04720; origin xyz=-0.0469 0 0 rpy=1.5708 0 -1.5708 -> xyz=0.00000 0.03559 0.00020
- joint FL3_joint: axis 0 0 1 -> 0.000 1.000 0.000; limit lower=-3 upper=3 effort=${effort_limit} velocity=3 -> lower=-2.35619 upper=-0.52360 effort=1.4 velocity=1.04720; origin xyz=0.1 0 0 rpy=0 0 0 -> xyz=0.00000 0.01071 -0.09996
- joint FL4_joint: axis 0 0 0 -> (none); origin xyz=0.094333 0 0 rpy=0 0 0 -> xyz=0.00000 -0.00834 -0.10000
- joint FR1_joint: axis 0 0 1 -> 1.000 0.000 0.000; limit lower=-3 upper=3 effort=${effort_limit} velocity=3 -> lower=-0.78540 upper=1.57080 effort=1.4 velocity=1.04720; origin xyz=0.0954 -0.04 0 rpy=1.5708 0 -1.5708 -> xyz=0.09170 -0.05355 -0.00279
- joint FR2_joint: axis 0 0 1 -> 0.000 1.000 0.000; limit lower=-3 upper=3 effort=${effort_limit} velocity=3 -> lower=0.00020 upper=2.35619 effort=1.4 velocity=1.04720; origin xyz=0.0469 0 0 rpy=1.5708 0 -1.5708 -> xyz=0.00000 -0.03559 0.00000
- joint FR3_joint: axis 0 0 1 -> 0.000 1.000 0.000; limit lower=-3 upper=3 effort=${effort_limit} velocity=3 -> lower=-2.35619 upper=-0.52360 effort=1.4 velocity=1.04720; origin xyz=0.1 0 0 rpy=0 0 0 -> xyz=0.00000 -0.01071 -0.09996
- joint FR4_joint: axis 0 0 0 -> (none); origin xyz=0.094333 0 0 rpy=0 0 0 -> xyz=0.00000 0.00834 -0.10000
- joint RL1_joint: axis 0 0 1 -> 1.000 0.000 0.000; limit lower=-3 upper=3 effort=${effort_limit} velocity=3 -> lower=-0.78540 upper=1.57080 effort=1.4 velocity=1.04720; origin xyz=-0.0954 0.04 0 rpy=1.5708 0 -1.5708 -> xyz=-0.09170 0.05355 -0.00279
- joint RL2_joint: axis 0 0 1 -> 0.000 1.000 0.000; limit lower=-3 upper=3 effort=${effort_limit} velocity=3 -> lower=0.00020 upper=2.35619 effort=1.4 velocity=1.04720; origin xyz=-0.0469 0 0 rpy=1.5708 0 -1.5708 -> xyz=0.00000 0.03559 0.00000
- joint RL3_joint: axis 0 0 1 -> 0.000 1.000 0.000; limit lower=-3 upper=3 effort=${effort_limit} velocity=3 -> lower=-2.35619 upper=-0.52360 effort=1.4 velocity=1.04720; origin xyz=0.1 0 0 rpy=0 0 0 -> xyz=0.00000 0.01071 -0.09996
- joint RL4_joint: axis 0 0 0 -> (none); origin xyz=0.094333 0 0 rpy=0 0 0 -> xyz=0.00000 -0.00834 -0.10000
- joint RR1_joint: axis 0 0 1 -> 1.000 0.000 0.000; limit lower=-3 upper=3 effort=${effort_limit} velocity=3 -> lower=-0.78540 upper=1.57080 effort=1.4 velocity=1.04720; origin xyz=-0.0954 -0.04 0 rpy=1.5708 0 -1.5708 -> xyz=-0.09170 -0.05355 -0.00279
- joint RR2_joint: axis 0 0 1 -> 0.000 1.000 0.000; limit lower=-3 upper=3 effort=${effort_limit} velocity=3 -> lower=0.00000 upper=2.35619 effort=1.4 velocity=1.04720; origin xyz=0.0469 0 0 rpy=1.5708 0 -1.5708 -> xyz=0.00000 -0.03559 0.00000
- joint RR3_joint: axis 0 0 1 -> 0.000 1.000 0.000; limit lower=-3 upper=3 effort=${effort_limit} velocity=3 -> lower=-2.35619 upper=-0.52360 effort=1.4 velocity=1.04720; origin xyz=0.1 0 0 rpy=0 0 0 -> xyz=0.00000 -0.01071 -0.09996
- joint RR4_joint: axis 0 0 0 -> (none); origin xyz=0.094333 0 0 rpy=0 0 0 -> xyz=0.00000 0.00834 -0.10000

Commit message: changed urdf

File: src/notspot_description/urdf/notspot.urdf (robot description, URDF)
Before this commit: robot notspot, 17 links, 16 joints
Links:
- link FL1: mass 0.34 -> 0.233
- link FL2: mass 0.084 -> 0.184
- link RL2: mass 0.084 -> 0.184
- link RR2: mass 0.084 -> 0.184

Commit message: Fixed axes

File: src/notspot_description/urdf/notspot.urdf (robot description, URDF)
Before this commit: robot notspot, 17 links, 16 joints
Joints:
- joint FL1_joint: axis 1.000 0.000 0.000 -> -1.000 0.000 0.000
- joint FR1_joint: axis 1.000 0.000 0.000 -> -1.000 0.000 0.000
- joint RL1_joint: axis 1.000 0.000 0.000 -> -1.000 0.000 0.000
- joint RR1_joint: axis 1.000 0.000 0.000 -> -1.000 0.000 0.000
